File: Hardware/HighBall_Hardware_v1/Avionics_Main_Board.sch (EAGLE design)
At the start: 17 parts

Commit message: Modifications to Spinner
Other:
- note added: "B"
- note removed: "A"
Changed lines of the file:
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@@
 <plain>
 <text x="149.86" y="25.4" size="5.08" layer="94">CONTROLLER AND I/O</text>
-<text x="238.76" y="5.08" size="5.08" layer="94">A</text>
+<text x="238.76" y="5.08" size="5.08" layer="94">B</text>
 </plain>
 <instances>
@@
 <text x="205.74" y="170.18" size="2.54" layer="94">Gas Valve (M-02)</text>
 <text x="165.1" y="170.18" size="2.54" layer="94">Ballast (M-01)</text>
-<text x="238.76" y="5.08" size="5.08" layer="94">A</text>
+<text x="238.76" y="5.08" size="5.08" layer="94">B</text>
 <text x="152.4" y="25.4" size="5.08" layer="94">POWER</text>
 </plain>
@@
 <wire x1="137.16" y1="78.74" x2="0" y2="78.74" width="0.1524" layer="94"/>
 <wire x1="137.16" y1="124.46" x2="137.16" y2="78.74" width="0.1524" layer="94"/>
-<text x="238.76" y="5.08" size="5.08" layer="94">A</text>
+<text x="238.76" y="5.08" size="5.08" layer="94">B</text>
 <text x="149.86" y="25.4" size="5.08" layer="94">INSTRUMENTATION</text>
 <text x="177.8" y="119.38" size="2.54" layer="94">Iridium / RockBLOCK Module</text>

Commit message: Code and Schematic Updates
Added State Machine .h & .cpp file
Added Resistor to LM335 and added battery voltage measurement to schematic.
Board Layout TBD
Parts:
- added R1: 2k, SparkFun-Resistors:1KOHM-HORIZ-1/4W-5%
- added R2: 20k, SparkFun-Resistors:1KOHM-HORIZ-1/4W-5%
- added R3: 130k, SparkFun-Resistors:1KOHM-HORIZ-1/4W-5%
Connections:
- new net VBAT_SENSE: C-1.A3, R2.1, R3.2
- net AGND: now also TIT-01.-; no longer TIT-01.ADJ
- net GND: now also R3.1
- net TIT-01: now also R1.2
- net VBAT: now also R2.2
- net VCC_1: now also R1.1; no longer TIT-01.-
Other:
- note added: "Battery Voltage"
Changed lines of the file:
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@@
 <?xml version="1.0" encoding="utf-8"?>
 <!DOCTYPE eagle SYSTEM "eagle.dtd">
-<eagle version="9.1.1">
+<eagle version="9.1.2">
 <drawing>
 <settings>
@@
 <part name="GND17" library="SparkFun-PowerSymbols" library_urn="urn:adsk.eagle:library:530" deviceset="GND" device=""/>
 <part name="SUPPLY13" library="SparkFun-PowerSymbols" library_urn="urn:adsk.eagle:library:530" deviceset="VCC_1" device=""/>
+<part name="R1" library="SparkFun-Resistors" library_urn="urn:adsk.eagle:library:532" deviceset="1KOHM" device="-HORIZ-1/4W-5%" package3d_urn="urn:adsk.eagle:package:39658/1" value="2k"/>
+<part name="GND18" library="SparkFun-PowerSymbols" library_urn="urn:adsk.eagle:library:530" deviceset="GND" device=""/>
+<part name="R2" library="SparkFun-Resistors" library_urn="urn:adsk.eagle:library:532" deviceset="1KOHM" device="-HORIZ-1/4W-5%" package3d_urn="urn:adsk.eagle:package:39658/1" value="20k"/>
+<part name="R3" library="SparkFun-Resistors" library_urn="urn:adsk.eagle:library:532" deviceset="1KOHM" device="-HORIZ-1/4W-5%" package3d_urn="urn:adsk.eagle:package:39658/1" value="130k"/>
 </parts>
 <sheets>
@@
 <wire x1="195.58" y1="137.16" x2="200.66" y2="137.16" width="0.1524" layer="91"/>
 <label x="198.12" y="137.16" size="1.778" layer="95"/>
+</segment>
+</net>
+<net name="VBAT_SENSE" class="0">
+<segment>
+<pinref part="C-1" gate="G$1" pin="A3"/>
+<wire x1="160.02" y1="142.24" x2="154.94" y2="142.24" width="0.1524" layer="91"/>
+<label x="142.24" y="142.24" size="1.778" layer="95"/>
 </segment>
 </net>
@@
 <text x="55.88" y="114.3" size="2.54" layer="94">GPS-01</text>
 <text x="50.8" y="111.76" size="1.778" layer="94">I2C Address: 0x10</text>
-<wire x1="137.16" y1="78.74" x2="0" y2="78.74" width="0.1524" layer="94"/>
+<wire x1="137.16" y1="78.74" x2="99.06" y2="78.74" width="0.1524" layer="94"/>
+<wire x1="99.06" y1="78.74" x2="0" y2="78.74" width="0.1524" layer="94"/>
 <wire x1="137.16" y1="124.46" x2="137.16" y2="78.74" width="0.1524" layer="94"/>
 <text x="238.76" y="5.08" size="5.08" layer="94">B</text>
@@
 <text x="177.8" y="119.38" size="2.54" layer="94">Iridium / RockBLOCK Module</text>
 <wire x1="137.16" y1="78.74" x2="248.92" y2="78.74" width="0.1524" layer="94"/>
+<wire x1="99.06" y1="78.74" x2="99.06" y2="0" width="0.1524" layer="94"/>
+<text x="33.02" y="73.66" size="2.54" layer="94">Battery Voltage</text>
 </plain>
 <instances>
 <instance part="TIT-01" gate="G$1" x="96.52" y="154.94"/>
-<instance part="U$3" gate="G$1" x="109.22" y="144.78"/>
-<instance part="SUPPLY3" gate="G$2" x="99.06" y="147.32" rot="R90"/>
+<instance part="U$3" gate="G$1" x="93.98" y="147.32" rot="R270"/>
+<instance part="SUPPLY3" gate="G$2" x="104.14" y="132.08" rot="R180"/>
 <instance part="FRAME2" gate="G$1" x="0" y="0"/>
 <instance part="FRAME2" gate="G$2" x="147.32" y="0"/>
@@
 <instance part="GND17" gate="1" x="180.34" y="86.36"/>
 <instance part="SUPPLY13" gate="G$2" x="180.34" y="93.98"/>
+<instance part="R1" gate="G$1" x="104.14" y="139.7" rot="R90"/>
+<instance part="GND18" gate="1" x="45.72" y="27.94"/>
+<instance part="R2" gate="G$1" x="45.72" y="53.34" rot="R90"/>
+<instance part="R3" gate="G$1" x="45.72" y="38.1" rot="R90"/>
 </instances>
 <busses>
@@
 <net name="VCC_1" class="0">
 <segment>
-<pinref part="TIT-01" gate="G$1" pin="-"/>
-<pinref part="SUPPLY3" gate="G$2" pin="VCC_1"/>
-<wire x1="99.06" y1="149.86" x2="99.06" y2="147.32" width="0.1524" layer="91"/>
-</segment>
-<segment>
 <pinref part="IMU-01" gate="G$1" pin="VBAT"/>
 <wire x1="25.4" y1="160.02" x2="12.7" y2="160.02" width="0.1524" layer="91"/>
@@
 <wire x1="200.66" y1="93.98" x2="180.34" y2="93.98" width="0.1524" layer="91"/>
 </segment>
-</net>
-<net name="AGND" class="0">
-<segment>
-<pinref part="U$3" gate="G$1" pin="AGND"/>
-<pinref part="TIT-01" gate="G$1" pin="ADJ"/>
-<wire x1="109.22" y1="147.32" x2="109.22" y2="149.86" width="0.1524" layer="91"/>
-</segment>
-</net>
-<net name="TIT-01" class="0">
-<segment>
-<pinref part="TIT-01" gate="G$1" pin="+"/>
-<wire x1="104.14" y1="149.86" x2="104.14" y2="147.32" width="0.1524" layer="91"/>
-<label x="101.6" y="149.86" size="1.778" layer="95" rot="R270"/>
+<segment>
+<pinref part="SUPPLY3" gate="G$2" pin="VCC_1"/>
+<pinref part="R1" gate="G$1" pin="1"/>
+<wire x1="104.14" y1="132.08" x2="104.14" y2="134.62" width="0.1524" layer="91"/>
 </segment>
 </net>
@@
 <wire x1="200.66" y1="88.9" x2="180.34" y2="88.9" width="0.1524" layer="91"/>
 </segment>
+<segment>
+<pinref part="GND18" gate="1" pin="GND"/>
+<pinref part="R3" gate="G$1" pin="1"/>
+<wire x1="45.72" y1="30.48" x2="45.72" y2="33.02" width="0.1524" layer="91"/>
+</segment>
 </net>
 <net name="VCC_2" class="0">
@@
 </segment>
 </net>
+<net name="AGND" class="0">
+<segment>
+<pinref part="TIT-01" gate="G$1" pin="-"/>
+<wire x1="99.06" y1="149.86" x2="99.06" y2="147.32" width="0.1524" layer="91"/>
+<pinref part="U$3" gate="G$1" pin="AGND"/>
+<wire x1="99.06" y1="147.32" x2="96.52" y2="147.32" width="0.1524" layer="91"/>
+</segment>
+</net>
+<net name="TIT-01" class="0">
+<segment>
+<pinref part="R1" gate="G$1" pin="2"/>
+<pinref part="TIT-01" gate="G$1" pin="+"/>
+<wire x1="104.14" y1="144.78" x2="104.14" y2="147.32" width="0.1524" layer="91"/>
+<wire x1="104.14" y1="147.32" x2="104.14" y2="149.86" width="0.1524" layer="91"/>
+<wire x1="104.14" y1="147.32" x2="114.3" y2="147.32" width="0.1524" layer="91"/>
+<junction x="104.14" y="147.32"/>
+<label x="109.22" y="147.32" size="1.778" layer="95"/>
+</segment>
+</net>
+<net name="VBAT" class="0">
+<segment>
+<pinref part="R2" gate="G$1" pin="2"/>
+<wire x1="45.72" y1="58.42" x2="45.72" y2="60.96" width="0.1524" layer="91"/>
+<wire x1="45.72" y1="60.96" x2="40.64" y2="60.96" width="0.1524" layer="91"/>
+<label x="35.56" y="60.96" size="2.54" layer="95"/>
+</segment>
+</net>
+<net name="VBAT_SENSE" class="0">
+<segment>
+<pinref part="R2" gate="G$1" pin="1"/>
+<pinref part="R3" gate="G$1" pin="2"/>
+<wire x1="45.72" y1="48.26" x2="45.72" y2="45.72" width="0.1524" layer="91"/>
+<wire x1="45.72" y1="45.72" x2="45.72" y2="43.18" width="0.1524" layer="91"/>
+<wire x1="45.72" y1="45.72" x2="53.34" y2="45.72" width="0.1524" layer="91"/>
+<junction x="45.72" y="45.72"/>
+<label x="50.8" y="45.72" size="2.54" layer="95"/>
+</segment>
+</net>

Commit message: Schematic Rev C and CAD Files changes
Completed rev C of hardware schematic
Created new PCB layout
Updated tolerance on ballast dispenser
Connections:
- removed net N$3: M-01.1
- removed net N$4: M-01.2
- removed net N$6: M-02.2
- removed net N$7: M-02.1
- net GND: now also M-01.1, M-02.1
- net VCC_1: now also M-01.2, M-02.2
Other:
- note added: "C"
- note removed: "B"
Changed lines of the file:
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@@
 <?xml version="1.0" encoding="utf-8"?>
 <!DOCTYPE eagle SYSTEM "eagle.dtd">
-<eagle version="9.1.2">
+<eagle version="9.1.3">
 <drawing>
 <settings>
@@
 <plain>
 <text x="149.86" y="25.4" size="5.08" layer="94">CONTROLLER AND I/O</text>
-<text x="238.76" y="5.08" size="5.08" layer="94">B</text>
+<text x="238.76" y="5.08" size="5.08" layer="94">C</text>
 </plain>
 <instances>
@@
 <text x="205.74" y="170.18" size="2.54" layer="94">Gas Valve (M-02)</text>
 <text x="165.1" y="170.18" size="2.54" layer="94">Ballast (M-01)</text>
-<text x="238.76" y="5.08" size="5.08" layer="94">B</text>
 <text x="152.4" y="25.4" size="5.08" layer="94">POWER</text>
+<text x="238.76" y="5.08" size="5.08" layer="94">C</text>
 </plain>
 <instances>
@@
 <pinref part="Q-02" gate="NMOS" pin="S"/>
 </segment>
+<segment>
+<wire x1="172.72" y1="157.48" x2="172.72" y2="160.02" width="0.1524" layer="91"/>
+<pinref part="GND12" gate="1" pin="GND"/>
+<pinref part="M-01" gate="J$1" pin="1"/>
+<wire x1="175.26" y1="157.48" x2="172.72" y2="157.48" width="0.1524" layer="91"/>
+</segment>
+<segment>
+<wire x1="213.36" y1="157.48" x2="213.36" y2="160.02" width="0.1524" layer="91"/>
+<pinref part="GND13" gate="1" pin="GND"/>
+<pinref part="M-02" gate="J$1" pin="1"/>
+<wire x1="215.9" y1="157.48" x2="213.36" y2="157.48" width="0.1524" layer="91"/>
+</segment>
 </net>
 <net name="VCC_1" class="0">
@@
 <wire x1="58.42" y1="167.64" x2="63.5" y2="167.64" width="0.1524" layer="91"/>
 <pinref part="SUPPLY1" gate="G$2" pin="VCC_1"/>
+</segment>
+<segment>
+<pinref part="M-01" gate="J$1" pin="2"/>
+<wire x1="175.26" y1="154.94" x2="170.18" y2="154.94" width="0.1524" layer="91"/>
+<pinref part="SUPPLY8" gate="G$2" pin="VCC_1"/>
+</segment>
+<segment>
+<pinref part="M-02" gate="J$1" pin="2"/>
+<wire x1="215.9" y1="154.94" x2="213.36" y2="154.94" width="0.1524" layer="91"/>
+<wire x1="213.36" y1="154.94" x2="210.82" y2="154.94" width="0.1524" layer="91"/>
+<pinref part="SUPPLY9" gate="G$2" pin="VCC_1"/>
 </segment>
 </net>
@@
 </segment>
 </net>
-<net name="N$3" class="0">
-<segment>
-<pinref part="M-01" gate="J$1" pin="1"/>
-<wire x1="175.26" y1="157.48" x2="172.72" y2="157.48" width="0.1524" layer="91"/>
-<wire x1="172.72" y1="157.48" x2="172.72" y2="160.02" width="0.1524" layer="91"/>
-<pinref part="GND12" gate="1" pin="GND"/>
-</segment>
-</net>
-<net name="N$4" class="0">
-<segment>
-<pinref part="M-01" gate="J$1" pin="2"/>
-<wire x1="175.26" y1="154.94" x2="170.18" y2="154.94" width="0.1524" layer="91"/>
-<pinref part="SUPPLY8" gate="G$2" pin="VCC_1"/>
-</segment>
-</net>
 <net name="M-01" class="0">
 <segment>
@@
 <wire x1="213.36" y1="152.4" x2="210.82" y2="152.4" width="0.1524" layer="91"/>
 <label x="210.82" y="152.4" size="1.778" layer="95"/>
-</segment>
-</net>
-<net name="N$6" class="0">
-<segment>
-<pinref part="M-02" gate="J$1" pin="2"/>
-<wire x1="215.9" y1="154.94" x2="213.36" y2="154.94" width="0.1524" layer="91"/>
-<wire x1="213.36" y1="154.94" x2="210.82" y2="154.94" width="0.1524" layer="91"/>
-<pinref part="SUPPLY9" gate="G$2" pin="VCC_1"/>
-</segment>
-</net>
-<net name="N$7" class="0">
-<segment>
-<pinref part="M-02" gate="J$1" pin="1"/>
-<wire x1="215.9" y1="157.48" x2="213.36" y2="157.48" width="0.1524" layer="91"/>
-<wire x1="213.36" y1="157.48" x2="213.36" y2="160.02" width="0.1524" layer="91"/>
-<pinref part="GND13" gate="1" pin="GND"/>
 </segment>
 </net>
@@
 <wire x1="99.06" y1="78.74" x2="0" y2="78.74" width="0.1524" layer="94"/>
 <wire x1="137.16" y1="124.46" x2="137.16" y2="78.74" width="0.1524" layer="94"/>
-<text x="238.76" y="5.08" size="5.08" layer="94">B</text>
 <text x="149.86" y="25.4" size="5.08" layer="94">INSTRUMENTATION</text>
 <text x="177.8" y="119.38" size="2.54" layer="94">Iridium / RockBLOCK Module</text>
@@
 <wire x1="99.06" y1="78.74" x2="99.06" y2="0" width="0.1524" layer="94"/>
 <text x="33.02" y="73.66" size="2.54" layer="94">Battery Voltage</text>
+<text x="238.76" y="5.08" size="5.08" layer="94">C</text>
 </plain>
 <instances>

Commit message: Electrical board changes
Parts:
- added COMM-02: (no value), SparkFun-Connectors:CONN_03LOCK
- R2: value 20k -> 18k
- R3: value 130k -> 150k
Connections:
- net N$1 renamed HE-01_OUT
- net N$2 renamed HE-02_OUT
- new net COMM-02-RX: C-1.1(TX0), COMM-02.1
- new net COMM-02-TX: C-1.0(RX0), COMM-02.2
- net GND: now also COMM-02.3
Other:
- note added: "BATTERY VOLTAGE"
- note added: "SERIAL COMM"
- note removed: "Battery Voltage"
- moved on the sheet: R2, R3
Changed lines of the file:
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@@
 </variantdefs>
 <classes>
-<class number="0" name="default" width="0.508" drill="0.508">
-<clearance class="0" value="0.254"/>
+<class number="0" name="default" width="0.635" drill="0.899159375">
+<clearance class="0" value="0.381"/>
+</class>
+<class number="1" name="power" width="1.016" drill="0.899159375">
+<clearance class="1" value="0.762"/>
 </class>
 </classes>
@@
 <part name="R1" library="SparkFun-Resistors" library_urn="urn:adsk.eagle:library:532" deviceset="1KOHM" device="-HORIZ-1/4W-5%" package3d_urn="urn:adsk.eagle:package:39658/1" value="2k"/>
 <part name="GND18" library="SparkFun-PowerSymbols" library_urn="urn:adsk.eagle:library:530" deviceset="GND" device=""/>
-<part name="R2" library="SparkFun-Resistors" library_urn="urn:adsk.eagle:library:532" deviceset="1KOHM" device="-HORIZ-1/4W-5%" package3d_urn="urn:adsk.eagle:package:39658/1" value="20k"/>
-<part name="R3" library="SparkFun-Resistors" library_urn="urn:adsk.eagle:library:532" deviceset="1KOHM" device="-HORIZ-1/4W-5%" package3d_urn="urn:adsk.eagle:package:39658/1" value="130k"/>
+<part name="R2" library="SparkFun-Resistors" library_urn="urn:adsk.eagle:library:532" deviceset="1KOHM" device="-HORIZ-1/4W-5%" package3d_urn="urn:adsk.eagle:package:39658/1" value="18k"/>
+<part name="R3" library="SparkFun-Resistors" library_urn="urn:adsk.eagle:library:532" deviceset="1KOHM" device="-HORIZ-1/4W-5%" package3d_urn="urn:adsk.eagle:package:39658/1" value="150k"/>
+<part name="COMM-02" library="SparkFun-Connectors" library_urn="urn:adsk.eagle:library:513" deviceset="CONN_03" device="LOCK" package3d_urn="urn:adsk.eagle:package:38071/1"/>
 </parts>
 <sheets>
@@
 </segment>
 </net>
-<net name="VCC_1" class="0">
+<net name="VCC_1" class="1">
 <segment>
 <pinref part="SUPPLY5" gate="G$2" pin="VCC_1"/>
@@
 </segment>
 </net>
-<net name="VCC_2" class="0">
+<net name="VCC_2" class="1">
 <segment>
 <pinref part="SUPPLY7" gate="G$1" pin="VCC_2"/>
@@
 <wire x1="160.02" y1="142.24" x2="154.94" y2="142.24" width="0.1524" layer="91"/>
 <label x="142.24" y="142.24" size="1.778" layer="95"/>
+</segment>
+</net>
+<net name="COMM-02-TX" class="0">
+<segment>
+<pinref part="C-1" gate="G$1" pin="0(RX0)"/>
+<wire x1="160.02" y1="109.22" x2="154.94" y2="109.22" width="0.1524" layer="91"/>
+<label x="144.78" y="109.22" size="1.778" layer="95"/>
+</segment>
+</net>
+<net name="COMM-02-RX" class="0">
+<segment>
+<pinref part="C-1" gate="G$1" pin="1(TX0)"/>
+<wire x1="160.02" y1="106.68" x2="154.94" y2="106.68" width="0.1524" layer="91"/>
+<label x="144.78" y="106.68" size="1.778" layer="95"/>
 </segment>
 </net>
@@
 </busses>
 <nets>
-<net name="VBAT" class="0">
+<net name="VBAT" class="1">
 <segment>
 <pinref part="VR-01" gate="G$1" pin="IN+"/>
@@
 </segment>
 </net>
-<net name="VCC_1" class="0">
+<net name="VCC_1" class="1">
 <segment>
 <pinref part="VR-01" gate="G$1" pin="OUT+"/>
@@
 </segment>
 </net>
-<net name="VCC_2" class="0">
+<net name="VCC_2" class="1">
 <segment>
 <pinref part="VR-02" gate="G$1" pin="OUT+"/>
@@
 </segment>
 </net>
-<net name="N$1" class="0">
+<net name="HE-01_OUT" class="1">
 <segment>
 <wire x1="93.98" y1="154.94" x2="93.98" y2="157.48" width="0.1524" layer="91"/>
@@
 </segment>
 </net>
-<net name="N$2" class="0">
+<net name="HE-02_OUT" class="1">
 <segment>
 <wire x1="127" y1="154.94" x2="127" y2="157.48" width="0.1524" layer="91"/>
@@
 <text x="55.88" y="114.3" size="2.54" layer="94">GPS-01</text>
 <text x="50.8" y="111.76" size="1.778" layer="94">I2C Address: 0x10</text>
-<wire x1="137.16" y1="78.74" x2="99.06" y2="78.74" width="0.1524" layer="94"/>
-<wire x1="99.06" y1="78.74" x2="0" y2="78.74" width="0.1524" layer="94"/>
+<wire x1="137.16" y1="78.74" x2="63.5" y2="78.74" width="0.1524" layer="94"/>
+<wire x1="63.5" y1="78.74" x2="0" y2="78.74" width="0.1524" layer="94"/>
 <wire x1="137.16" y1="124.46" x2="137.16" y2="78.74" width="0.1524" layer="94"/>
 <text x="149.86" y="25.4" size="5.08" layer="94">INSTRUMENTATION</text>
 <text x="177.8" y="119.38" size="2.54" layer="94">Iridium / RockBLOCK Module</text>
 <wire x1="137.16" y1="78.74" x2="248.92" y2="78.74" width="0.1524" layer="94"/>
-<wire x1="99.06" y1="78.74" x2="99.06" y2="0" width="0.1524" layer="94"/>
-<text x="33.02" y="73.66" size="2.54" layer="94">Battery Voltage</text>
+<wire x1="63.5" y1="78.74" x2="63.5" y2="0" width="0.1524" layer="94"/>
+<text x="17.78" y="71.12" size="2.54" layer="94">BATTERY VOLTAGE</text>
 <text x="238.76" y="5.08" size="5.08" layer="94">C</text>
+<wire x1="137.16" y1="78.74" x2="137.16" y2="0" width="0.1524" layer="94"/>
+<text x="88.9" y="71.12" size="2.54" layer="94">SERIAL COMM</text>
 </plain>
 <instances>
@@
 <instance part="SUPPLY13" gate="G$2" x="180.34" y="93.98"/>
 <instance part="R1" gate="G$1" x="104.14" y="139.7" rot="R90"/>
-<instance part="GND18" gate="1" x="45.72" y="27.94"/>
-<instance part="R2" gate="G$1" x="45.72" y="53.34" rot="R90"/>
-<instance part="R3" gate="G$1" x="45.72" y="38.1" rot="R90"/>
+<instance part="GND18" gate="1" x="30.48" y="25.4"/>
+<instance part="R2" gate="G$1" x="30.48" y="50.8" rot="R90"/>
+<instance part="R3" gate="G$1" x="30.48" y="35.56" rot="R90"/>
+<instance part="COMM-02" gate="J$1" x="127" y="48.26" rot="R180"/>
 </instances>
 <busses>
 </busses>
 <nets>
-<net name="VCC_1" class="0">
+<net name="VCC_1" class="1">
 <segment>
 <pinref part="IMU-01" gate="G$1" pin="VBAT"/>
@@
 <pinref part="GND18" gate="1" pin="GND"/>
 <pinref part="R3" gate="G$1" pin="1"/>
-<wire x1="45.72" y1="30.48" x2="45.72" y2="33.02" width="0.1524" layer="91"/>
-</segment>
-</net>
-<net name="VCC_2" class="0">
+<wire x1="30.48" y1="27.94" x2="30.48" y2="30.48" width="0.1524" layer="91"/>
+</segment>
+<segment>
+<pinref part="COMM-02" gate="J$1" pin="3"/>
+<wire x1="119.38" y1="45.72" x2="114.3" y2="45.72" width="0.1524" layer="91"/>
+<label x="114.3" y="45.72" size="1.778" layer="95"/>
+</segment>
+</net>
+<net name="VCC_2" class="1">
 <segment>
 <pinref part="PIT-01" gate="G$1" pin="3V3"/>
@@
 </segment>
 </net>
-<net name="VBAT" class="0">
+<net name="VBAT" class="1">
 <segment>
 <pinref part="R2" gate="G$1" pin="2"/>
-<wire x1="45.72" y1="58.42" x2="45.72" y2="60.96" width="0.1524" layer="91"/>
-<wire x1="45.72" y1="60.96" x2="40.64" y2="60.96" width="0.1524" layer="91"/>
-<label x="35.56" y="60.96" size="2.54" layer="95"/>
+<wire x1="30.48" y1="55.88" x2="30.48" y2="58.42" width="0.1524" layer="91"/>
+<wire x1="30.48" y1="58.42" x2="25.4" y2="58.42" width="0.1524" layer="91"/>
+<label x="20.32" y="58.42" size="2.54" layer="95"/>
 </segment>
 </net>
@@
 <pinref part="R2" gate="G$1" pin="1"/>
 <pinref part="R3" gate="G$1" pin="2"/>
-<wire x1="45.72" y1="48.26" x2="45.72" y2="45.72" width="0.1524" layer="91"/>
-<wire x1="45.72" y1="45.72" x2="45.72" y2="43.18" width="0.1524" layer="91"/>
-<wire x1="45.72" y1="45.72" x2="53.34" y2="45.72" width="0.1524" layer="91"/>
-<junction x="45.72" y="45.72"/>
-<label x="50.8" y="45.72" size="2.54" layer="95"/>
+<wire x1="30.48" y1="45.72" x2="30.48" y2="43.18" width="0.1524" layer="91"/>
+<wire x1="30.48" y1="43.18" x2="30.48" y2="40.64" width="0.1524" layer="91"/>
+<wire x1="30.48" y1="43.18" x2="38.1" y2="43.18" width="0.1524" layer="91"/>
+<junction x="30.48" y="43.18"/>
+<label x="35.56" y="43.18" size="2.54" layer="95"/>
+</segment>
+</net>
+<net name="COMM-02-RX" class="0">
+<segment>
+<pinref part="COMM-02" gate="J$1" pin="1"/>
+<wire x1="119.38" y1="50.8" x2="114.3" y2="50.8" width="0.1524" layer="91"/>
+<label x="104.14" y="50.8" size="1.778" layer="95"/>
+</segment>
+</net>
+<net name="COMM-02-TX" class="0">
+<segment>
+<pinref part="COMM-02" gate="J$1" pin="2"/>
+<wire x1="119.38" y1="48.26" x2="114.3" y2="48.26" width="0.1524" layer="91"/>
+<label x="104.14" y="48.26" size="1.778" layer="95"/>
 </segment>
 </net>
@@
 </sheet>
 </sheets>
-<errors>
-</errors>
 </schematic>
 </drawing>

Commit message: Electronics and Hardware changes
Parts:
- removed R1: 2k, SparkFun-Resistors:1KOHM-HORIZ-1/4W-5%
- COMM-02: device SparkFun-Connectors:CONN_03LOCK -> SparkFun-Connectors:CONN_05LOCK
- R3: value 150k -> 15k
Connections:
- net COMM-02-RX renamed COMM-02-TXO
- net COMM-02-TX renamed COMM-02-RXI
- new net 5V: TIT-01.ADJ
- net GND: now also COMM-02.5; no longer COMM-02.3
- net TIT-01: no longer R1.2
- net VCC_1: no longer R1.1
